File: pcb/pcb.kicad_sch (KiCad schematic)
At the start: 2 parts, among them U1 ATmega16U4-A

Commit message: save pcb
Parts:
- added D10, D11, D12, D13, D14, D15, D16, D17, D18, D19, D2, D20, D21, D22, D23, D24, D25, D26, D27, D28, D29, D3, D30, D31, D32, D33, D34, D35, D36, D37, D38, D39, D4, D40, D41, D42, D43, D44, D45, D46, D47, D48, D49, D5, D50, D51, D52, D53, D54, D55, D56, D57, D58, D59, D6, D60, D7, D8, D9: 1N5817, Diode_THT:D_DO-41_SOD81_P10.16mm_Horizontal, symbol Diode:1N5817
- added SW1, SW10, SW11, SW12, SW13, SW14, SW15, SW16, SW17, SW18, SW19, SW2, SW20, SW21, SW22, SW23, SW24, SW25, SW26, SW27, SW28, SW29, SW3, SW30, SW31, SW32, SW33, SW34, SW35, SW36, SW37, SW38, SW39, SW4, SW40, SW41, SW42, SW43, SW44, SW45, SW46, SW47, SW48, SW49, SW5, SW50, SW51, SW52, SW53, SW54, SW55, SW56, SW57, SW58, SW59, SW6, SW60, SW7, SW8, SW9: SW_SPST, symbol Switch:SW_SPST
Connections:
- net c1l: now reaches D1.1 (K)
- net c1l: now also D2.1 (K), D3.1 (K), D4.1 (K), D5.1 (K)
- net at D1.2 (A): now also SW1.2 (B)
- net GNDPWR: now reaches U1.15 (GND), U1.23 (GND), U1.35 (GND), U1.43 (GND)
- new net: D38.2 (A), SW38.2 (B)
- new net: D52.2 (A), SW52.2 (B)
- new net: D55.2 (A), SW55.2 (B)
- new net: D43.2 (A), SW43.2 (B)
- new net: D5.2 (A), SW5.2 (B)
- new net: D58.2 (A), SW58.2 (B)
- new net: D9.2 (A), SW9.2 (B)
- new net: D12.2 (A), SW12.2 (B)
- new net: D33.2 (A), SW33.2 (B)
- new net: D7.2 (A), SW7.2 (B)
- new net: D31.2 (A), SW31.2 (B)
- new net: D3.2 (A), SW3.2 (B)
- new net: D11.2 (A), SW11.2 (B)
- new net: D36.2 (A), SW36.2 (B)
- new net: D21.2 (A), SW21.2 (B)
- new net: D16.2 (A), SW16.2 (B)
- new net: D35.2 (A), SW35.2 (B)
- new net: D41.2 (A), SW41.2 (B)
- new net: D6.2 (A), SW6.2 (B)
- new net: D37.2 (A), SW37.2 (B)
- new net: D13.2 (A), SW13.2 (B)
- new net: D42.2 (A), SW42.2 (B)
- new net: D28.2 (A), SW28.2 (B)
- new net: D50.2 (A), SW50.2 (B)
- new net: D24.2 (A), SW24.2 (B)
- new net: D20.2 (A), SW20.2 (B)
- new net: D32.2 (A), SW32.2 (B)
- new net: D46.2 (A), SW46.2 (B)
- new net: D34.2 (A), SW34.2 (B)
- new net: D49.2 (A), SW49.2 (B)
- new net: D25.2 (A), SW25.2 (B)
- new net: D48.2 (A), SW48.2 (B)
- new net: D15.2 (A), SW15.2 (B)
- new net: D14.2 (A), SW14.2 (B)
- new net: D45.2 (A), SW45.2 (B)
- new net: D22.2 (A), SW22.2 (B)
- new net: D56.2 (A), SW56.2 (B)
- new net: D57.2 (A), SW57.2 (B)
- new net: D18.2 (A), SW18.2 (B)
- new net: D47.2 (A), SW47.2 (B)
- new net: D10.2 (A), SW10.2 (B)
- new net: D17.2 (A), SW17.2 (B)
- new net: D53.2 (A), SW53.2 (B)
- new net: D39.2 (A), SW39.2 (B)
- new net: D19.2 (A), SW19.2 (B)
- new net: D51.2 (A), SW51.2 (B)
- new net: D44.2 (A), SW44.2 (B)
- new net: D23.2 (A), SW23.2 (B)
- new net: D40.2 (A), SW40.2 (B)
- new net: D26.2 (A), SW26.2 (B)
- new net: D8.2 (A), SW8.2 (B)
- new net: D29.2 (A), SW29.2 (B)
- new net: D2.2 (A), SW2.2 (B)
- new net: D4.2 (A), SW4.2 (B)
- new net: D30.2 (A), SW30.2 (B)
- new net: D54.2 (A), SW54.2 (B)
- new net: D59.2 (A), SW59.2 (B)
- new net: D27.2 (A), SW27.2 (B)
- new net: D60.2 (A), SW60.2 (B)
- new net c1r: D12.1 (K), D18.1 (K), D24.1 (K), D30.1 (K), D6.1 (K)
- new net c2l: D10.1 (K), D11.1 (K), D7.1 (K), D8.1 (K), D9.1 (K)
- new net c2r: D36.1 (K), D37.1 (K), D38.1 (K), D39.1 (K), D40.1 (K)
- new net c3l: D13.1 (K), D14.1 (K), D15.1 (K), D16.1 (K), D17.1 (K)
- new net c3r: D41.1 (K), D42.1 (K), D43.1 (K), D44.1 (K), D45.1 (K)
- new net c4l: D19.1 (K), D20.1 (K), D21.1 (K), D22.1 (K), D23.1 (K)
- new net c4r: D46.1 (K), D47.1 (K), D48.1 (K), D49.1 (K), D50.1 (K)
- new net c5l: D25.1 (K), D26.1 (K), D27.1 (K), D28.1 (K), D29.1 (K)
- new net c5r: D51.1 (K), D52.1 (K), D53.1 (K), D54.1 (K), D55.1 (K)
- new net c6l: D31.1 (K), D32.1 (K), D33.1 (K), D34.1 (K), D35.1 (K)
- new net c6r: D56.1 (K), D57.1 (K), D58.1 (K), D59.1 (K), D60.1 (K)
- new net r1l: SW1.1 (A), SW13.1 (A), SW19.1 (A), SW25.1 (A), SW31.1 (A), SW7.1 (A)
- new net r1r: SW36.1 (A), SW41.1 (A), SW46.1 (A), SW51.1 (A), SW56.1 (A), SW6.1 (A)
- new net r2l: SW14.1 (A), SW2.1 (A), SW20.1 (A), SW26.1 (A), SW32.1 (A), SW8.1 (A)
- new net r2r: SW12.1 (A), SW37.1 (A), SW42.1 (A), SW47.1 (A), SW52.1 (A), SW57.1 (A)
- new net r3l: SW15.1 (A), SW21.1 (A), SW27.1 (A), SW3.1 (A), SW33.1 (A), SW9.1 (A)
- new net r3r: SW18.1 (A), SW38.1 (A), SW43.1 (A), SW48.1 (A), SW53.1 (A), SW58.1 (A)
- new net r4l: SW10.1 (A), SW16.1 (A), SW22.1 (A), SW28.1 (A), SW34.1 (A), SW4.1 (A)
- new net r4r: SW24.1 (A), SW39.1 (A), SW44.1 (A), SW49.1 (A), SW54.1 (A), SW59.1 (A)
- new net r5l: SW11.1 (A), SW17.1 (A), SW23.1 (A), SW29.1 (A), SW35.1 (A), SW5.1 (A)
- new net r5r: SW30.1 (A), SW40.1 (A), SW45.1 (A), SW50.1 (A), SW55.1 (A), SW60.1 (A)
Other:
- moved on the sheet: U1

Commit message: sanity save
Parts:
- removed D10: 1N5817, Diode_THT:D_DO-41_SOD81_P10.16mm_Horizontal, symbol Diode:1N5817
- added C1, C3: 100nF, symbol Device:C
- added C2, C4: 10µF, symbol Device:C
- added C5, C6: 1µF, symbol Device:C
- added D61, D62, D63, D64: 1N5817, Diode_THT:D_DO-41_SOD81_P10.16mm_Horizontal, symbol Diode:1N5817
- added P1, P2: USB_C_Plug_USB2.0, symbol Connector:USB_C_Plug_USB2.0
- added R1, R2, R3, R4: 22, symbol Device:R
- added R5, R6: 5100, symbol Device:R
- added SW61, SW62, SW63, SW64: SW_SPST, symbol Switch:SW_SPST
- added U2: ATmega16U4-A, Package_QFP:TQFP-44_10x10mm_P0.8mm, symbol MCU_Microchip_ATmega:ATmega16U4-A
Connections:
- net GNDPWR is gone; now on net GNDPWRL: U1.15 (GND), U1.23 (GND), U1.35 (GND), U1.43 (GND)
- net r4l is gone; now on net r3l: SW10.1 (A), SW16.1 (A), SW22.1 (A), SW28.1 (A), SW34.1 (A), SW4.1 (A)
- net c1l: now also D7.1 (K), D8.1 (K), D9.1 (K), U1.19 (PD1); no longer D1.1 (K), D2.1 (K), D3.1 (K), D4.1 (K), D5.1 (K)
- net c1r: now also D36.1 (K), D37.1 (K), D38.1 (K), U2.19 (PD1); no longer D12.1 (K), D18.1 (K), D24.1 (K), D6.1 (K)
- net c2l: now also D13.1 (K), D14.1 (K), D15.1 (K), D16.1 (K), U1.20 (PD2); no longer D11.1 (K), D7.1 (K), D8.1 (K), D9.1 (K)
- net c2r: now also D41.1 (K), D42.1 (K), U2.20 (PD2); no longer D36.1 (K), D37.1 (K), D38.1 (K)
- net c3l: now also D19.1 (K), D20.1 (K), D21.1 (K), D22.1 (K), U1.21 (PD3); no longer D13.1 (K), D14.1 (K), D15.1 (K), D16.1 (K), D17.1 (K)
- net c3r: now also D46.1 (K), U2.21 (PD3); no longer D41.1 (K), D42.1 (K)
- net c4l: now also D25.1 (K), D26.1 (K), D27.1 (K), D28.1 (K), U1.25 (PD4); no longer D19.1 (K), D20.1 (K), D21.1 (K), D22.1 (K), D23.1 (K)
- net c4r: now also U2.25 (PD4); no longer D46.1 (K)
- net c5l: now also D31.1 (K), D32.1 (K), D33.1 (K), D34.1 (K), U1.22 (PD5); no longer D25.1 (K), D26.1 (K), D27.1 (K), D28.1 (K), D29.1 (K)
- net c5r: now also U2.22 (PD5); no longer D55.1 (K)
- net c6l: now also D11.1 (K), D17.1 (K), D23.1 (K), D5.1 (K), U1.26 (PD6); no longer D31.1 (K), D32.1 (K), D33.1 (K), D34.1 (K), D35.1 (K)
- net c6r: now also D55.1 (K), U2.26 (PD6); no longer D59.1 (K), D60.1 (K)
- net r1l: now also SW11.1 (A), SW14.1 (A), SW2.1 (A), SW20.1 (A), SW26.1 (A), SW32.1 (A), SW35.1 (A), SW8.1 (A), U1.9 (PB1); no longer SW1.1 (A), SW13.1 (A), SW19.1 (A), SW25.1 (A), SW31.1 (A), SW7.1 (A)
- net r1r: now also SW12.1 (A), SW40.1 (A), SW44.1 (A), SW48.1 (A), SW52.1 (A), SW60.1 (A), U2.9 (PB1); no longer SW41.1 (A), SW46.1 (A), SW51.1 (A), SW6.1 (A)
- net r2l: now also SW15.1 (A), SW17.1 (A), SW21.1 (A), SW27.1 (A), SW3.1 (A), SW33.1 (A), SW9.1 (A), U1.10 (PB2), SW61.1 (A); no longer SW14.1 (A), SW2.1 (A), SW20.1 (A), SW26.1 (A), SW32.1 (A), SW8.1 (A)
- net r2r: now also SW18.1 (A), SW41.1 (A), SW45.1 (A), SW49.1 (A), SW53.1 (A), SW63.1 (A), U2.10 (PB2); no longer SW12.1 (A), SW42.1 (A), SW47.1 (A), SW52.1 (A)
- net r3l: now also SW23.1 (A), U1.11 (PB3), SW62.1 (A); no longer SW15.1 (A), SW21.1 (A), SW27.1 (A), SW3.1 (A), SW33.1 (A), SW9.1 (A)
- net r3r: now also SW24.1 (A), SW42.1 (A), SW46.1 (A), SW50.1 (A), SW54.1 (A), SW64.1 (A), U2.11 (PB3); no longer SW18.1 (A), SW43.1 (A), SW48.1 (A), SW53.1 (A)
- net c0l: now reaches U1.18 (PD0)
- net c0l: now also D1.1 (K), D2.1 (K), D3.1 (K), D4.1 (K)
- net c7l: now reaches U1.27 (PD7)
- net c7l: now also D29.1 (K), D35.1 (K), D61.1 (K), D62.1 (K)
- net D-l: now reaches U1.3 (D-)
- net D-l: now also R1.2
- net D+l: now reaches U1.4 (D+)
- net D+l: now also R2.2
- net GNDPWRL: now reaches U1.5 (UGND)
- net GNDPWRL: now also C1.2, C2.2, C5.2, P1.A1 (GND), P1.A12 (GND), P1.B1 (GND), P1.B12 (GND), R5.2
- net at U1.6 (UCAP): now also C5.1
- net VCCL: now reaches U1.7 (VBUS)
- net VCCL: now also C1.1, C2.1, P1.A4 (VBUS), P1.A9 (VBUS), P1.B4 (VBUS), P1.B9 (VBUS)
- net r0l: now reaches U1.8 (PB0)
- net r0l: now also SW1.1 (A), SW13.1 (A), SW19.1 (A), SW25.1 (A), SW29.1 (A), SW31.1 (A), SW5.1 (A), SW7.1 (A)
- removed net r4r: SW24.1 (A), SW39.1 (A), SW44.1 (A), SW49.1 (A), SW54.1 (A), SW59.1 (A)
- removed net r5l: SW11.1 (A), SW17.1 (A), SW23.1 (A), SW29.1 (A), SW35.1 (A), SW5.1 (A)
- removed net r5r: SW30.1 (A), SW40.1 (A), SW45.1 (A), SW50.1 (A), SW55.1 (A), SW60.1 (A)
- new net: D63.2 (A), SW63.2 (B)
- new net: P1.A7 (D-), R1.1
- new net: P2.A5 (CC), R6.1
- new net: C6.1, U2.6 (UCAP)
- new net: P1.A5 (CC), R5.1
- new net: D62.2 (A), SW62.2 (B)
- new net: P1.A6 (D+), R2.1
- new net: D64.2 (A), SW64.2 (B)
- new net: P2.A6 (D+), R4.1
- new net: D61.2 (A), SW61.2 (B)
- new net: U2.14 (VCC), U2.34 (VCC)
- new net: U2.24 (AVCC), U2.44 (AVCC)
- new net: P2.A7 (D-), R3.1
- new net D+r: R4.2, U2.4 (D+)
- new net D-r: R3.2, U2.3 (D-)
- new net GNDPWRR: C3.2, C4.2, C6.2, P2.A1 (GND), P2.A12 (GND), P2.B1 (GND), P2.B12 (GND), R6.2, U2.15 (GND), U2.23 (GND), U2.35 (GND), U2.43 (GND), U2.5 (UGND)
- new net VCCR: C3.1, C4.1, P2.A4 (VBUS), P2.A9 (VBUS), P2.B4 (VBUS), P2.B9 (VBUS), U2.7 (VBUS)
- new net c0r: D12.1 (K), D18.1 (K), D24.1 (K), D6.1 (K), U2.18 (PD0)
- new net c7r: D59.1 (K), D60.1 (K), D63.1 (K), D64.1 (K), U2.27 (PD7)
- new net r0r: SW30.1 (A), SW39.1 (A), SW43.1 (A), SW47.1 (A), SW51.1 (A), SW55.1 (A), SW59.1 (A), SW6.1 (A), U2.8 (PB0)
Other:
- moved on the sheet: U1

Commit message: updad
Parts:
- removed C5: 1µF, symbol Device:C
- removed R1, R2: 22, symbol Device:R
- removed R5: 5100, symbol Device:R
- added P3: R to L, symbol Connector:USB_C_Plug_USB2.0
- P1: value USB_C_Plug_USB2.0 -> L to R
- P2: value USB_C_Plug_USB2.0 -> R to computer
Connections:
- net GNDPWRL: no longer P1.A1 (GND), P1.A12 (GND), P1.B1 (GND), P1.B12 (GND)
- net GNDPWRR: now also P1.A1 (GND), P1.A12 (GND), P1.B1 (GND), P1.B12 (GND), P3.A1 (GND), P3.A12 (GND), P3.B1 (GND), P3.B12 (GND)
- net VCCL: no longer P1.A4 (VBUS), P1.A9 (VBUS), P1.B4 (VBUS), P1.B9 (VBUS), U1.7 (VBUS)
- net VCCR: now also P1.A4 (VBUS), P1.A9 (VBUS), P1.B4 (VBUS), P1.B9 (VBUS), U1.14 (VCC), U1.34 (VCC), U2.14 (VCC), U2.34 (VCC), P3.A4 (VBUS), P3.A9 (VBUS), P3.B4 (VBUS), P3.B9 (VBUS)
- net c0l: now also U1.8 (PB0); no longer U1.18 (PD0)
- net c0r: now also U2.8 (PB0); no longer U2.18 (PD0)
- net c1l: now also U1.9 (PB1); no longer U1.19 (PD1)
- net c1r: now also U2.9 (PB1); no longer U2.19 (PD1)
- net c2l: now also U1.10 (PB2); no longer U1.20 (PD2)
- net c2r: now also U2.10 (PB2); no longer U2.20 (PD2)
- net c3l: now also U1.11 (PB3); no longer U1.21 (PD3)
- net c3r: now also U2.11 (PB3); no longer U2.21 (PD3)
- net c4l: now also U1.28 (PB4); no longer U1.25 (PD4)
- net c4r: now also U2.28 (PB4); no longer U2.25 (PD4)
- net c5l: now also U1.29 (PB5); no longer U1.22 (PD5)
- net c5r: now also U2.29 (PB5); no longer U2.22 (PD5)
- net c6l: now also U1.30 (PB6); no longer U1.26 (PD6)
- net c6r: now also U2.30 (PB6); no longer U2.26 (PD6)
- net c7l: now also U1.12 (PB7); no longer U1.27 (PD7)
- net c7r: now also U2.12 (PB7); no longer U2.27 (PD7)
- net r0l: now also U1.39 (PF4); no longer U1.8 (PB0)
- net r0r: now also U2.39 (PF4); no longer U2.8 (PB0)
- net r1l: now also U1.38 (PF5); no longer U1.9 (PB1)
- net r1r: now also U2.38 (PF5); no longer U2.9 (PB1)
- net r2l: now also U1.37 (PF6); no longer U1.10 (PB2)
- net r2r: now also U2.37 (PF6); no longer U2.10 (PB2)
- net r3l: now also U1.36 (PF7); no longer U1.11 (PB3)
- net r3r: now also U2.36 (PF7); no longer U2.11 (PB3)
- net TX: now reaches P1.A7 (D-)
- net TX: now also U1.20 (PD2), U2.21 (PD3), P3.A7 (D-)
- net RX: now reaches P1.A6 (D+)
- net RX: now also U1.21 (PD3), U2.20 (PD2), P3.A6 (D+)
- net D+l: no longer names the net of U1.4 (D+)
- net D-l: no longer names the net of U1.3 (D-)
Other:
- moved on the sheet: C6, U2

Commit message: fx
Connections:
- net VCCL: now also P1.A4 (VBUS), P1.A9 (VBUS), P1.B4 (VBUS), P1.B9 (VBUS)
- net VCCR: no longer P1.A4 (VBUS), P1.A9 (VBUS), P1.B4 (VBUS), P1.B9 (VBUS)
Changed lines of the file:
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@@
 			)
 		)
-		(property "Value" "VCCR"
+		(property "Value" "VCCL"
 			(at 278.13 152.4 0)
 			(effects

Commit message: upd and add switches submodule
Parts:
- C1, C2, C3, C4, C6: footprint (none) -> Capacitor_SMD:C_1206_3216Metric_Pad1.33x1.80mm_HandSolder
- P1: footprint (none) -> Connector_USB:USB_C_Plug_JAE_DX07P024AJ1
- P2, P3: footprint (none) -> Connector_USB:USB_C_Plug_Molex_105444
- R3, R4, R6: footprint (none) -> Resistor_SMD:R_1206_3216Metric_Pad1.30x1.75mm_HandSolder
Changed lines of the file:
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@@
 			)
 		)
-		(property "Footprint" ""
+		(property "Footprint" "Resistor_SMD:R_1206_3216Metric_Pad1.30x1.75mm_HandSolder"
 			(at 355.6 166.878 90)
 			(show_name yes)
@@
 			)
 		)
-		(property "Footprint" ""
+		(property "Footprint" "Capacitor_SMD:C_1206_3216Metric_Pad1.33x1.80mm_HandSolder"
 			(at 390.8552 96.52 0)
 			(effects
@@
 			)
 		)
-		(property "Footprint" ""
+		(property "Footprint" "Connector_USB:USB_C_Plug_Molex_105444"
 			(at 300.99 176.53 0)
 			(effects
@@
 			)
 		)
-		(property "Footprint" ""
+		(property "Footprint" "Capacitor_SMD:C_1206_3216Metric_Pad1.33x1.80mm_HandSolder"
 			(at 390.8552 187.96 0)
 			(effects
@@
 			)
 		)
-		(property "Footprint" ""
+		(property "Footprint" "Capacitor_SMD:C_1206_3216Metric_Pad1.33x1.80mm_HandSolder"
 			(at 375.6152 161.29 0)
 			(effects
@@
 			)
 		)
-		(property "Footprint" ""
+		(property "Footprint" "Capacitor_SMD:C_1206_3216Metric_Pad1.33x1.80mm_HandSolder"
 			(at 375.6152 187.96 0)
 			(effects
@@
 			)
 		)
-		(property "Footprint" ""
+		(property "Footprint" "Resistor_SMD:R_1206_3216Metric_Pad1.30x1.75mm_HandSolder"
 			(at 355.6 179.578 90)
 			(effects
@@
 			)
 		)
-		(property "Footprint" ""
+		(property "Footprint" "Capacitor_SMD:C_1206_3216Metric_Pad1.33x1.80mm_HandSolder"
 			(at 390.8552 161.29 0)
 			(effects
@@
 			)
 		)
-		(property "Footprint" ""
+		(property "Footprint" "Connector_USB:USB_C_Plug_JAE_DX07P024AJ1"
 			(at 261.62 176.53 0)
 			(effects
@@
 			)
 		)
-		(property "Footprint" ""
+		(property "Footprint" "Resistor_SMD:R_1206_3216Metric_Pad1.30x1.75mm_HandSolder"
 			(at 355.6 174.498 90)
 			(effects
@@
 			)
 		)
-		(property "Footprint" ""
+		(property "Footprint" "Connector_USB:USB_C_Plug_Molex_105444"
 			(at 340.36 175.26 0)
 			(effects

Commit message: upd
Parts:
- removed C6: 1µF, Capacitor_SMD:C_1206_3216Metric_Pad1.33x1.80mm_HandSolder, symbol Device:C
- removed P2: R to computer, Connector_USB:USB_C_Plug_Molex_105444, symbol Connector:USB_C_Plug_USB2.0
- removed R3, R4: 22, Resistor_SMD:R_1206_3216Metric_Pad1.30x1.75mm_HandSolder, symbol Device:R
- removed R6: 5100, Resistor_SMD:R_1206_3216Metric_Pad1.30x1.75mm_HandSolder, symbol Device:R
- removed U1, U2: ATmega16U4-A, Package_QFP:TQFP-44_10x10mm_P0.8mm, symbol MCU_Microchip_ATmega:ATmega16U4-A
- added U1, U2: RP2040-ZERO, RP2040-ZERO:MODULE_RP2040-ZERO, symbol RP2040:RP2040-ZERO
- SW1, SW10, SW11, SW12, SW13, SW14, SW15, SW16, SW17, SW18, SW19, SW2, SW20, SW21, SW22, SW23, SW24, SW25, SW26, SW27, SW28, SW29, SW3, SW30, SW31, SW32, SW33, SW34, SW35, SW36, SW37, SW38, SW39, SW4, SW40, SW41, SW42, SW43, SW44, SW45, SW46, SW47, SW48, SW49, SW5, SW50, SW51, SW52, SW53, SW54, SW55, SW56, SW57, SW58, SW59, SW6, SW60, SW61, SW62, SW63, SW64, SW7, SW8, SW9: footprint (none) -> Footprints:SW_MX_THT

Commit message: updates
Parts:
- added D10: 1N5817, Diode_THT:D_DO-41_SOD81_P10.16mm_Horizontal, symbol Diode:1N5817
- added R1, R2: 4700, Resistor_SMD:R_1206_3216Metric_Pad1.30x1.75mm_HandSolder, symbol Device:R
- SW1, SW10, SW11, SW12, SW13, SW14, SW15, SW16, SW17, SW18, SW19, SW2, SW20, SW21, SW22, SW23, SW24, SW25, SW26, SW27, SW28, SW29, SW3, SW30, SW31, SW32, SW33, SW34, SW35, SW36, SW37, SW38, SW39, SW4, SW40, SW41, SW42, SW43, SW44, SW45, SW46, SW47, SW48, SW49, SW5, SW50, SW51, SW52, SW53, SW54, SW55, SW56, SW57, SW58, SW59, SW6, SW60, SW61, SW62, SW63, SW64, SW7, SW8, SW9: footprint Footprints:SW_MX_THT -> Keyboard Footprints:SW_MX_THT_nSilk
- U1, U2: footprint RP2040-ZERO:MODULE_RP2040-ZERO -> rp2040:MODULE_RP2040-ZERO
Connections:
- net RX is gone; now on net SDA: P1.A6 (D+), P3.A6 (D+)
- net TX is gone; now on net SCL: P1.A7 (D-), P3.A7 (D-)
- net VCCL: now also U1.23 (5V), R1.1, R2.1
- net VCCR: now also U2.23 (5V)
- net c0l: now also U1.1 (GP0)
- net c0r: now also U2.8 (GP7)
- net c1l: now also U1.2 (GP1), D10.1 (K)
- net c1r: now also U2.7 (GP6)
- net c2l: now also U1.3 (GP2)
- net c2r: now also U2.6 (GP5)
- net c3l: now also U1.4 (GP3)
- net c3r: now also U2.5 (GP4)
- net c4l: now also U1.5 (GP4)
- net c4r: now also U2.4 (GP3)
- net c5l: now also U1.6 (GP5)
- net c5r: now also U2.3 (GP2)
- net c6l: now also U1.7 (GP6)
- net c6r: now also U2.2 (GP1)
- net c7l: now also U1.8 (GP7)
- net c7r: now also U2.1 (GP0)
- net r0l: now also U1.16 (GP15)
- net r0r: now also U2.13 (GP12)
- net r1l: now also U1.15 (GP14)
- net r1r: now also U2.14 (GP13)
- net r2l: now also U1.14 (GP13)
- net r2r: now also U2.15 (GP14)
- net r3l: now also U1.13 (GP12)
- net r3r: now also U2.16 (GP15)
- net at SW10.2 (B): now also D10.2 (A)
- net SDA: now reaches U1.17 (GP26)
- net SDA: now also U2.17 (GP26), R2.2
- net SCL: now reaches U1.18 (GP27)
- net SCL: now also U2.18 (GP27), R1.2
- net GNDPWR: now reaches U1.22 (GND)
- net GNDPWR: now also U2.22 (GND)
- no-connect marks 0 -> 20
Other:
- moved on the sheet: C1, C2, C3, C4, P1, P3, U1, U2

Commit message: a lot of updates
Parts:
- removed P3: R to L, Connector_USB:USB_C_Plug_Molex_105444, symbol Connector:USB_C_Plug_USB2.0
- added P2: R to L, Connector_USB:USB_C_Plug_JAE_DX07P024AJ1, symbol Connector:USB_C_Plug_USB2.0
Connections:
- net GNDPWRL: now also P1.A1 (GND), P1.A12 (GND), P1.B1 (GND), P1.B12 (GND), U1.22 (GND)
- net GNDPWRR: now also U2.22 (GND), P2.A1 (GND), P2.A12 (GND), P2.B1 (GND), P2.B12 (GND); no longer P1.A1 (GND), P1.A12 (GND), P1.B1 (GND), P1.B12 (GND)
- net SCL: now also P2.A7 (D-)
- net SDA: now also P2.A6 (D+)
- net VCCR: now also P2.A4 (VBUS), P2.A9 (VBUS), P2.B4 (VBUS), P2.B9 (VBUS)
- removed net GNDPWR: U1.22 (GND), U2.22 (GND)
Changed lines of the file:
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@@
 			)
 		)
-		(property "Value" "GNDPWR"
+		(property "Value" "GNDPWRR"
 			(at 374.523 69.85 0)
 			(effects
@@
 			)
 		)
-		(property "Value" "GNDPWR"
+		(property "Value" "GNDPWRL"
 			(at 304.673 67.31 0)
 			(effects
@@
 	)
 	(symbol
-		(lib_id "Diode:1N5817")
-		(at 152.4 36.83 90)
+		(lib_id "Connector:USB_C_Plug_USB2.0")
+		(at 304.8 110.49 0)
 		(unit 1)
 		(exclude_from_sim no)
@@
 		(dnp no)
 		(fields_autoplaced yes)
-		(property "Reference" "D30"
-			(at 154.94 35.8774 90)
+		(property "Reference" "P2"
+			(at 304.8 87.63 0)
 			(effects
 				(font
 					(size 1.27 1.27)
 				)
-				(justify right)
-				(hide yes)
 			)
 		)
-		(property "Value" "1N5817"
-			(at 154.94 38.4174 90)
+		(property "Value" "R to L"
+			(at 304.8 90.17 0)
 			(effects
 				(font
 					(size 1.27 1.27)
 				)
-				(justify right)
-				(hide yes)
 			)
 		)
-		(property "Footprint" "Diode_THT:D_DO-41_SOD81_P10.16mm_Horizontal"
-			(at 156.845 36.83 0)
+		(property "Footprint" "Connector_USB:USB_C_Plug_JAE_DX07P024AJ1"
+			(at 308.61 110.49 0)
 			(effects
 				(font
@@
 			)
 		)
-		(property "Datasheet" "http://www.vishay.com/docs/88525/1n5817.pdf"
-			(at 152.4 36.83 0)
+		(property "Datasheet" "https://www.usb.org/sites/default/files/documents/usb_type-c.zip"
+			(at 308.61 110.49 0)
 			(effects
 				(font
@@
 			)
 		)
-		(property "Description" "20V 1A Schottky Barrier Rectifier Diode, DO-41"
-			(at 152.4 36.83 0)
+		(property "Description" "USB 2.0-only Type-C Plug connector"
+			(at 304.8 110.49 0)
 			(effects
 				(font
@@
 			)
 		)
-		(pin "2"
+		(pin "A1"
 		)
-		(pin "1"
+		(pin "A12"
+		)
+		(pin "A6"
+		)
+		(pin "A7"
+		)
+		(pin "A9"
+		)
+		(pin "B1"
+		)
+		(pin "B12"
+		)
+		(pin "B4"
+		)
+		(pin "B5"
+		)
+		(pin "B9"
+		)
+		(pin "S1"
+		)
+		(pin "A5"
+		)
+		(pin "A4"
 		)
 		(instances
 			(project "pcb"
 				(path "/bd59a313-a6de-4d3b-8b64-7b9522a3d186"
-					(reference "D30")
+					(reference "P2")
 					(unit 1)
 				)
@@
 	)
 	(symbol
-		(lib_id "Connector:USB_C_Plug_USB2.0")
-		(at 304.8 110.49 0)
+		(lib_id "Diode:1N5817")
+		(at 152.4 36.83 90)
 		(unit 1)
 		(exclude_from_sim no)
@@
 		(dnp no)
 		(fields_autoplaced yes)
-		(property "Reference" "P3"
-			(at 304.8 87.63 0)
+		(property "Reference" "D30"
+			(at 154.94 35.8774 90)
 			(effects
 				(font
 					(size 1.27 1.27)
 				)
+				(justify right)
+				(hide yes)
 			)
 		)
-		(property "Value" "R to L"
-			(at 304.8 90.17 0)
+		(property "Value" "1N5817"
+			(at 154.94 38.4174 90)
 			(effects
 				(font
 					(size 1.27 1.27)
 				)
+				(justify right)
+				(hide yes)
 			)
 		)
-		(property "Footprint" "Connector_USB:USB_C_Plug_Molex_105444"
-			(at 308.61 110.49 0)
+		(property "Footprint" "Diode_THT:D_DO-41_SOD81_P10.16mm_Horizontal"
+			(at 156.845 36.83 0)
 			(effects
 				(font
@@
 			)
 		)
-		(property "Datasheet" "https://www.usb.org/sites/default/files/documents/usb_type-c.zip"
-			(at 308.61 110.49 0)
+		(property "Datasheet" "http://www.vishay.com/docs/88525/1n5817.pdf"
+			(at 152.4 36.83 0)
 			(effects
 				(font
@@
 			)
 		)
-		(property "Description" "USB 2.0-only Type-C Plug connector"
-			(at 304.8 110.49 0)
+		(property "Description" "20V 1A Schottky Barrier Rectifier Diode, DO-41"
+			(at 152.4 36.83 0)
 			(effects
 				(font
@@
 			)
 		)
-		(pin "A1"
-		)
-		(pin "B5"
-		)
-		(pin "B4"
-		)
-		(pin "B1"
-		)
-		(pin "A4"
-		)
-		(pin "A7"
-		)
-		(pin "A9"
-		)
-		(pin "A12"
-		)
-		(pin "A5"
-		)
-		(pin "S1"
-		)
-		(pin "B12"
-		)
-		(pin "A6"
+		(pin "2"
 		)
-		(pin "B9"
+		(pin "1"
 		)
 		(instances
 			(project "pcb"
 				(path "/bd59a313-a6de-4d3b-8b64-7b9522a3d186"
-					(reference "P3")
+					(reference "D30")
 					(unit 1)
 				)
@@
 			)
 		)
-		(property "Value" "GNDPWRR"
+		(property "Value" "GNDPWRL"
 			(at 265.303 137.16 0)
 			(effects
