File: pcb/pcb.kicad_sch (KiCad schematic)
At the start: 138 parts, among them P1 L to R, P2 R to L, SW1 SW_SPST, SW10 SW_SPST, SW11 SW_SPST, SW12 SW_SPST, SW13 SW_SPST, SW14 SW_SPST, SW15 SW_SPST, SW16 SW_SPST, SW17 SW_SPST, SW18 SW_SPST, SW19 SW_SPST, SW2 SW_SPST, SW20 SW_SPST, SW21 SW_SPST, SW22 SW_SPST, SW23 SW_SPST, SW24 SW_SPST, SW25 SW_SPST, SW26 SW_SPST, SW27 SW_SPST, SW28 SW_SPST, SW29 SW_SPST, SW3 SW_SPST, SW30 SW_SPST, SW31 SW_SPST, SW32 SW_SPST, SW33 SW_SPST, SW34 SW_SPST, SW35 SW_SPST, SW36 SW_SPST, SW37 SW_SPST, SW38 SW_SPST, SW39 SW_SPST, SW4 SW_SPST, SW40 SW_SPST, SW41 SW_SPST, SW42 SW_SPST, SW43 SW_SPST, SW44 SW_SPST, SW45 SW_SPST, SW46 SW_SPST, SW47 SW_SPST, SW48 SW_SPST, SW49 SW_SPST, SW5 SW_SPST, SW50 SW_SPST, SW51 SW_SPST, SW52 SW_SPST, SW53 SW_SPST, SW54 SW_SPST, SW55 SW_SPST, SW56 SW_SPST, SW57 SW_SPST, SW58 SW_SPST, SW59 SW_SPST, SW6 SW_SPST, SW60 SW_SPST, SW61 SW_SPST, SW62 SW_SPST, SW63 SW_SPST, SW64 SW_SPST, SW7 SW_SPST, SW8 SW_SPST, SW9 SW_SPST, U1 RP2040-ZERO, U2 RP2040-ZERO

Commit message: lfgooooo
Connections:
- net VCCL: no longer R1.1
- net VCCR: now also R1.1
- net c0r: now also U2.1 (GP0); no longer U2.8 (GP7)
- net c1r: now also U2.2 (GP1); no longer U2.7 (GP6)
- net c2r: now also U2.3 (GP2); no longer U2.6 (GP5)
- net c3r: now also U2.4 (GP3); no longer U2.5 (GP4)
- net c4r: now also U2.5 (GP4); no longer U2.4 (GP3)
- net c5r: now also U2.6 (GP5); no longer U2.3 (GP2)
- net c6r: now also U2.7 (GP6); no longer U2.2 (GP1)
- net c7r: now also U2.8 (GP7); no longer U2.1 (GP0)

Commit message: think it si there
Parts:
- P1, P2: footprint Connector_USB:USB_C_Plug_JAE_DX07P024AJ1 -> Connector_USB:USB_C_Receptacle_GCT_USB4085
Changed lines of the file:
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@@
 			)
 		)
-		(property "Footprint" "Connector_USB:USB_C_Plug_JAE_DX07P024AJ1"
+		(property "Footprint" "Connector_USB:USB_C_Receptacle_GCT_USB4085"
 			(at 308.61 110.49 0)
 			(effects
@@
 			)
 		)
-		(property "Footprint" "Connector_USB:USB_C_Plug_JAE_DX07P024AJ1"
+		(property "Footprint" "Connector_USB:USB_C_Receptacle_GCT_USB4085"
 			(at 269.24 110.49 0)
 			(effects

Commit message: to low prof
Parts:
- SW1, SW10, SW11, SW12, SW13, SW14, SW15, SW16, SW17, SW18, SW19, SW2, SW20, SW21, SW22, SW23, SW24, SW25, SW26, SW27, SW28, SW29, SW3, SW30, SW31, SW32, SW33, SW34, SW35, SW36, SW37, SW38, SW39, SW4, SW40, SW41, SW42, SW43, SW44, SW45, SW46, SW47, SW48, SW49, SW5, SW50, SW51, SW52, SW53, SW54, SW55, SW56, SW57, SW58, SW59, SW6, SW60, SW61, SW62, SW63, SW64, SW7, SW8, SW9: footprint Keyboard Footprints:SW_MX_THT_nSilk -> Keyboard Footprints:SW_Kailh_Choc_V2_THT
