File: pcb/pcb.kicad_pcb (KiCad board)
At the start: 2 copper layers, 5 x 8.2 mm, 138 parts, among them P1 L to R, P3 R to L, SW1 SW_SPST, SW10 SW_SPST, SW11 SW_SPST, SW12 SW_SPST, SW13 SW_SPST, SW14 SW_SPST, SW15 SW_SPST, SW16 SW_SPST, SW17 SW_SPST, SW18 SW_SPST, SW19 SW_SPST, SW2 SW_SPST, SW20 SW_SPST, SW21 SW_SPST, SW22 SW_SPST, SW23 SW_SPST, SW24 SW_SPST, SW25 SW_SPST, SW26 SW_SPST, SW27 SW_SPST, SW28 SW_SPST, SW29 SW_SPST, SW3 SW_SPST, SW30 SW_SPST, SW31 SW_SPST, SW32 SW_SPST, SW33 SW_SPST, SW34 SW_SPST, SW35 SW_SPST, SW36 SW_SPST, SW37 SW_SPST, SW38 SW_SPST, SW39 SW_SPST, SW4 SW_SPST, SW40 SW_SPST, SW41 SW_SPST, SW42 SW_SPST, SW43 SW_SPST, SW44 SW_SPST, SW45 SW_SPST, SW46 SW_SPST, SW47 SW_SPST, SW48 SW_SPST, SW49 SW_SPST, SW5 SW_SPST, SW50 SW_SPST, SW51 SW_SPST, SW52 SW_SPST, SW53 SW_SPST, SW54 SW_SPST, SW55 SW_SPST, SW56 SW_SPST, SW57 SW_SPST, SW58 SW_SPST, SW59 SW_SPST, SW6 SW_SPST, SW60 SW_SPST, SW61 SW_SPST, SW62 SW_SPST, SW63 SW_SPST, SW64 SW_SPST, SW7 SW_SPST, SW8 SW_SPST, SW9 SW_SPST, U1 RP2040-ZERO, U2 RP2040-ZERO

Commit message: a lot of updates
Parts:
- removed P3: R to L, Connector_USB:USB_C_Plug_Molex_105444
- added P2: R to L, Connector_USB:USB_C_Plug_JAE_DX07P024AJ1, F.Cu at (280.3, 71.7)
- D12, D18, D24, D30, D36, D37, D38, D39, D40, D41, D42, D43, D44, D45, D46, D47, D48, D49, D50, D51, D52, D53, D54, D55, D56, D57, D58, D59, D6, D60, D63, D64: moved to F.Cu
- moved D59 420.7 mm to (361.2, 75.2)
- moved D55 400.0 mm to (353.3, 84.8)
- moved SW39 273.9 mm to (370.0, 112.8)
- moved D39 266.4 mm to (375.4, 122.7)
- moved SW30 265.5 mm to (349.9, 112.8)
- moved D18 264.5 mm to (335.4, 163.3)
- moved SW24 264.3 mm to (329.9, 173.5)
- moved SW36 260.6 mm to (349.9, 132.8)
- moved D30 258.1 mm to (355.3, 122.9)
- moved SW6 257.2 mm to (329.8, 113.0)
- moved SW18 256.4 mm to (329.9, 153.2)
- moved D24 256.3 mm to (335.3, 183.5)
- moved SW12 252.0 mm to (329.9, 133.1)
- moved SW51 251.9 mm to (476.9, 106.7)
- moved SW59 251.9 mm to (534.0, 106.7)
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Connections:
- P1 pad A1: GNDPWRR -> GNDPWRL
- P1 pad A12: GNDPWRR -> GNDPWRL
- P1 pad B1: GNDPWRR -> GNDPWRL
- P1 pad B12: GNDPWRR -> GNDPWRL
- U1 pad 22: GNDPWR -> GNDPWRL
- U2 pad 22: GNDPWR -> GNDPWRR
Routing:
- net VCCL: track 0.00 -> 39.3 mm
- net GNDPWRL: track 0.00 -> 25.1 mm
- net SDA: track 0.00 -> 23.9 mm
- net SCL: track 0.14 -> 21.8 mm
- net c5l: track 130.3 -> 142.1 mm
- net c0l: track 232.6 -> 244.4 mm
- net c6l: track 106.5 -> 118.3 mm
- net r1l: track 151.6 -> 163.4 mm
- net c3l: track 174.8 -> 185.8 mm
- net r0l: track 153.7 -> 164.7 mm
- net c4l: track 159.0 -> 169.8 mm
- net c2l: track 197.2 -> 206.5 mm
- net c1l: track 217.9 -> 224.9 mm
- net r2l: track 172.1 -> 176.7 mm
- net r3l: track 193.1 -> 197.7 mm
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Other:
- board size 5 x 8.2 mm -> 8.2 x 5 mm

Commit message: yooooo thankn you gpt
Parts:
- moved SW6 203.1 mm to (529.8, 77.5)
- moved SW24 203.0 mm to (529.7, 137.5)
- moved SW18 203.0 mm to (529.7, 117.5)
- moved SW12 202.9 mm to (529.7, 97.5)
- moved SW64 192.3 mm to (389.7, 137.5)
- moved SW38 182.0 mm to (509.7, 137.5)
- moved SW63 169.1 mm to (389.7, 117.5)
- moved SW30 163.8 mm to (509.8, 77.5)
- moved SW36 163.6 mm to (509.7, 97.5)
- moved SW58 159.4 mm to (409.7, 137.5)
- moved SW37 157.6 mm to (509.7, 117.5)
- moved SW60 153.7 mm to (389.7, 97.5)
- moved SW42 147.9 mm to (489.7, 137.5)
- moved SW59 147.2 mm to (389.7, 77.5)
- moved SW54 131.3 mm to (429.7, 137.5)
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Changed lines of the file:
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@@
 	(footprint "Keyboard Footprints:SW_MX_THT_nSilk"
 		(layer "F.Cu")
-		(at 505.46 106.68)
+		(at 409.819 77.500)
 		(descr "Cherry MX style mechanical keyboard switch, through-hole soldering, single-sided mounting.")
 		(tags "switch")
@@
 	(footprint "Keyboard Footprints:SW_MX_THT_nSilk"
 		(layer "F.Cu")
-		(at 448.31 106.68)
+		(at 449.739 77.500)
 		(descr "Cherry MX style mechanical keyboard switch, through-hole soldering, single-sided mounting.")
 		(tags "switch")
@@
 	(footprint "Keyboard Footprints:SW_MX_THT_nSilk"
 		(layer "F.Cu")
-		(at 426.259 256.019)
+		(at 469.739 137.500)
 		(descr "Cherry MX style mechanical keyboard switch, through-hole soldering, single-sided mounting.")
 		(tags "switch")
@@
 	(footprint "Keyboard Footprints:SW_MX_THT_nSilk"
 		(layer "F.Cu")
-		(at 426.259 192.494)
+		(at 469.739 117.500)
 		(descr "Cherry MX style mechanical keyboard switch, through-hole soldering, single-sided mounting.")
 		(tags "switch")
@@
 	(footprint "Keyboard Footprints:SW_MX_THT_nSilk"
 		(layer "F.Cu")
-		(at 511.259 192.494)
+		(at 409.739 117.500)
 		(descr "Cherry MX style mechanical keyboard switch, through-hole soldering, single-sided mounting.")
 		(tags "switch")
@@
 	(footprint "Keyboard Footprints:SW_MX_THT_nSilk"
 		(layer "F.Cu")
-		(at 541.259 192.494)
+		(at 389.659 117.500)
 		(descr "Cherry MX style mechanical keyboard switch, through-hole soldering, single-sided mounting.")
 		(tags "switch")
@@
 	(footprint "Keyboard Footprints:SW_MX_THT_nSilk"
 		(layer "F.Cu")
-		(at 329.946 153.162)
+		(at 529.739 117.500)
 		(descr "Cherry MX style mechanical keyboard switch, through-hole soldering, single-sided mounting.")
 		(tags "switch")
@@
 	(footprint "Keyboard Footprints:SW_MX_THT_nSilk"
 		(layer "F.Cu")
-		(at 349.885 132.842)
+		(at 509.659 97.500)
 		(descr "Cherry MX style mechanical keyboard switch, through-hole soldering, single-sided mounting.")
 		(tags "switch")
@@
 	(footprint "Keyboard Footprints:SW_MX_THT_nSilk"
 		(layer "F.Cu")
-		(at 538.099 137.414)
+		(at 389.659 97.500)
 		(descr "Cherry MX style mechanical keyboard switch, through-hole soldering, single-sided mounting.")
 		(tags "switch")
@@
 	(footprint "Keyboard Footprints:SW_MX_THT_nSilk"
 		(layer "F.Cu")
-		(at 534.035 106.68)
+		(at 389.739 77.500)
 		(descr "Cherry MX style mechanical keyboard switch, through-hole soldering, single-sided mounting.")
 		(tags "switch")
@@
 	(footprint "Keyboard Footprints:SW_MX_THT_nSilk"
 		(layer "F.Cu")
-		(at 541.179 256.019)
+		(at 389.739 137.500)
 		(descr "Cherry MX style mechanical keyboard switch, through-hole soldering, single-sided mounting.")
 		(tags "switch")
@@
 	(footprint "Keyboard Footprints:SW_MX_THT_nSilk"
 		(layer "F.Cu")
-		(at 476.885 106.68)
+		(at 429.739 77.500)
 		(descr "Cherry MX style mechanical keyboard switch, through-hole soldering, single-sided mounting.")
 		(tags "switch")
@@
 	(footprint "Keyboard Footprints:SW_MX_THT_nSilk"
 		(layer "F.Cu")
-		(at 371.179 255.519)
+		(at 509.739 137.500)
 		(descr "Cherry MX style mechanical keyboard switch, through-hole soldering, single-sided mounting.")
 		(tags "switch")
@@
 	(footprint "Keyboard Footprints:SW_MX_THT_nSilk"
 		(layer "F.Cu")
-		(at 395.224 137.414)
+		(at 489.659 97.500)
 		(descr "Cherry MX style mechanical keyboard switch, through-hole soldering, single-sided mounting.")
 		(tags "switch")
@@
 	(footprint "Keyboard Footprints:SW_MX_THT_nSilk"
 		(layer "F.Cu")
-		(at 329.946 133.096)
+		(at 529.659 97.500)
 		(descr "Cherry MX style mechanical keyboard switch, through-hole soldering, single-sided mounting.")
 		(tags "switch")
@@
 	(footprint "Keyboard Footprints:SW_MX_THT_nSilk"
 		(layer "F.Cu")
-		(at 419.735 106.68)
+		(at 469.739 77.500)
 		(descr "Cherry MX style mechanical keyboard switch, through-hole soldering, single-sided mounting.")
 		(tags "switch")
@@
 	(footprint "Keyboard Footprints:SW_MX_THT_nSilk"
 		(layer "F.Cu")
-		(at 371.179 192.494)
+		(at 509.739 117.500)
 		(descr "Cherry MX style mechanical keyboard switch, through-hole soldering, single-sided mounting.")
 		(tags "switch")
@@
 	(footprint "Keyboard Footprints:SW_MX_THT_nSilk"
 		(layer "F.Cu")
-		(at 349.885 112.776)
+		(at 509.819 77.500)
 		(descr "Cherry MX style mechanical keyboard switch, through-hole soldering, single-sided mounting.")
 		(tags "switch")
@@
 	(footprint "Keyboard Footprints:SW_MX_THT_nSilk"
 		(layer "F.Cu")
-		(at 452.374 137.414)
+		(at 449.659 97.500)
 		(descr "Cherry MX style mechanical keyboard switch, through-hole soldering, single-sided mounting.")
 		(tags "switch")
@@
 	(footprint "Keyboard Footprints:SW_MX_THT_nSilk"
 		(layer "F.Cu")
-		(at 486.259 256.019)
+		(at 429.739 137.500)
 		(descr "Cherry MX style mechanical keyboard switch, through-hole soldering, single-sided mounting.")
 		(tags "switch")
@@
 	(footprint "Keyboard Footprints:SW_MX_THT_nSilk"
 		(layer "F.Cu")
-		(at 509.524 137.414)
+		(at 409.739 97.500)
 		(descr "Cherry MX style mechanical keyboard switch, through-hole soldering, single-sided mounting.")
 		(tags "switch")
@@
 	(footprint "Keyboard Footprints:SW_MX_THT_nSilk"
 		(layer "F.Cu")
-		(at 329.819 113.03)
+		(at 529.819 77.500)
 		(descr "Cherry MX style mechanical keyboard switch, through-hole soldering, single-sided mounting.")
 		(tags "switch")
@@
 	(footprint "Keyboard Footprints:SW_MX_THT_nSilk"
 		(layer "F.Cu")
-		(at 396.259 192.494)
+		(at 489.739 117.500)
 		(descr "Cherry MX style mechanical keyboard switch, through-hole soldering, single-sided mounting.")
 		(tags "switch")
@@
 	(footprint "Keyboard Footprints:SW_MX_THT_nSilk"
 		(layer "F.Cu")
-		(at 456.259 192.494)
+		(at 449.659 117.500)
 		(descr "Cherry MX style mechanical keyboard switch, through-hole soldering, single-sided mounting.")
 		(tags "switch")
@@
 	(footprint "Keyboard Footprints:SW_MX_THT_nSilk"
 		(layer "F.Cu")
-		(at 456.179 256.019)
+		(at 449.739 137.500)
 		(descr "Cherry MX style mechanical keyboard switch, through-hole soldering, single-sided mounting.")
 		(tags "switch")
@@
 	(footprint "Keyboard Footprints:SW_MX_THT_nSilk"
 		(layer "F.Cu")
-		(at 329.946 173.482)
+		(at 529.739 137.500)
 		(descr "Cherry MX style mechanical keyboard switch, through-hole soldering, single-sided mounting.")
 		(tags "switch")
@@
 	(footprint "Keyboard Footprints:SW_MX_THT_nSilk"
 		(layer "F.Cu")
-		(at 516.259 256.019)
+		(at 409.659 137.500)
 		(descr "Cherry MX style mechanical keyboard switch, through-hole soldering, single-sided mounting.")
 		(tags "switch")
@@
 	(footprint "Keyboard Footprints:SW_MX_THT_nSilk"
 		(layer "F.Cu")
-		(at 369.951 112.776)
+		(at 489.739 77.500)
 		(descr "Cherry MX style mechanical keyboard switch, through-hole soldering, single-sided mounting.")
 		(tags "switch")
@@
 	(footprint "Keyboard Footprints:SW_MX_THT_nSilk"
 		(layer "F.Cu")
-		(at 401.339 256.019)
+		(at 489.739 137.500)
 		(descr "Cherry MX style mechanical keyboard switch, through-hole soldering, single-sided mounting.")
 		(tags "switch")
@@
 	(footprint "Keyboard Footprints:SW_MX_THT_nSilk"
 		(layer "F.Cu")
-		(at 480.949 137.414)
+		(at 429.739 97.500)
 		(descr "Cherry MX style mechanical keyboard switch, through-hole soldering, single-sided mounting.")
 		(tags "switch")
@@
 	(footprint "Keyboard Footprints:SW_MX_THT_nSilk"
 		(layer "F.Cu")
-		(at 481.179 192.494)
+		(at 429.659 117.500)
 		(descr "Cherry MX style mechanical keyboard switch, through-hole soldering, single-sided mounting.")
 		(tags "switch")
@@
 	(footprint "Keyboard Footprints:SW_MX_THT_nSilk"
 		(layer "F.Cu")
-		(at 423.799 137.414)
+		(at 469.659 97.500)
 		(descr "Cherry MX style mechanical keyboard switch, through-hole soldering, single-sided mounting.")
 		(tags "switch")

Commit message: lfgooooo
Parts:
- moved D64 299.5 mm to (283.7, 147.7), turned to 0 degrees
- moved D63 283.3 mm to (283.7, 127.6), turned to 0 degrees
- moved D60 259.6 mm to (283.8, 107.5), turned to 0 degrees
- moved D58 253.0 mm to (303.7, 147.6), turned to 0 degrees
- moved D57 237.6 mm to (303.7, 127.6), turned to 0 degrees
- moved D56 212.3 mm to (303.7, 107.5), turned to 0 degrees
- moved D54 211.6 mm to (323.7, 147.8), turned to 0 degrees
- moved D53 193.2 mm to (323.8, 127.6), turned to 0 degrees
- moved D51 183.5 mm to (323.8, 87.6), turned to 0 degrees
- moved D50 173.5 mm to (343.7, 147.7), turned to 0 degrees
- moved D52 165.6 mm to (323.8, 107.5), turned to 0 degrees
- moved D49 151.5 mm to (343.7, 127.6), turned to 0 degrees
- moved D46 142.9 mm to (363.7, 147.7), turned to 0 degrees
- moved D47 136.4 mm to (343.7, 87.6), turned to 0 degrees
- moved D42 125.7 mm to (383.7, 147.7), turned to 0 degrees
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Connections:
- R1 pad 1: VCCL -> VCCR
- U2 pad 1: c7r -> c0r
- U2 pad 2: c6r -> c1r
- U2 pad 3: c5r -> c2r
- U2 pad 4: c4r -> c3r
- U2 pad 5: c3r -> c4r
- U2 pad 6: c2r -> c5r
- U2 pad 7: c1r -> c6r
- U2 pad 8: c0r -> c7r
Routing:
- net c0r: track 0.00 -> 229.8 mm
- net r3r: track 0.00 -> 209.7 mm
- net c1r: track 0.00 -> 208.8 mm
- net r2r: track 0.00 -> 194.6 mm
- net r0r: track 0.00 -> 194.1 mm
- net c2r: track 0.00 -> 190.7 mm
- net r1r: track 0.00 -> 183.7 mm
- net c3r: track 0.00 -> 165.6 mm
- net c4r: track 0.00 -> 144.3 mm
- net c5r: track 0.00 -> 123.5 mm
- net c6r: track 0.00 -> 103.3 mm
- net c7r: track 0.00 -> 83.5 mm
- net SCL: track 21.8 -> 68.7 mm
- net VCCR: track 0.00 -> 41.2 mm
- net SDA: track 23.9 -> 63.3 mm
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
Commit message: think it si there
Parts:
- P1, P2: footprint Connector_USB:USB_C_Plug_JAE_DX07P024AJ1 -> Connector_USB:USB_C_Receptacle_GCT_USB4085
- moved P1 122.3 mm to (269.1, 179.4)
- moved P2 120.6 mm to (326.3, 179.4)
- moved U1 119.0 mm to (282.4, 189.0)
- moved C1 119.0 mm to (265.9, 186.8)
- moved C2 119.0 mm to (265.9, 182.8)
- moved D1 119.0 mm to (115.7, 193.9)
- moved D10 119.0 mm to (135.7, 253.9)
- moved D11 119.0 mm to (235.7, 213.9)
- moved D13 119.0 mm to (155.7, 193.9)
- moved D14 119.0 mm to (155.7, 213.9)
- moved D15 119.0 mm to (155.7, 233.9)
- moved D16 119.0 mm to (155.7, 253.9)
- moved D17 119.0 mm to (235.8, 233.9)
- moved D19 119.0 mm to (175.7, 193.9)
- moved D2 119.0 mm to (115.7, 213.9)
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Routing:
- net VCCL: track 70.5 -> 27.6 mm
- net GNDPWRL: track 25.1 -> 37.8 mm
- net VCCR: track 41.2 -> 46.3 mm
- net GNDPWRR: track 35.4 -> 40.1 mm
- net SCL: track 68.7 -> 65.8 mm
- net r3r: track 209.7 -> 212.3 mm
- net r2r: track 194.6 -> 195.8 mm
- net SDA: track 63.3 -> 62.3 mm
Other:
- board size 8.2 x 5 mm -> 386.1 x 84.1 mm

Commit message: qfx
Routing:
- net Net-(D58-A): track 0.00 -> 9.67 mm
- net Net-(D55-A): track 0.00 -> 9.66 mm
- net Net-(D56-A): track 0.00 -> 9.57 mm
- net c5l: track 142.1 -> 139.3 mm
- net c0l: track 244.4 -> 245.3 mm
Changed lines of the file:
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@@
 			(outputformat 1)
 			(mirror no)
-			(drillshape 1)
+			(drillshape 0)
 			(scaleselection 1)
 			(outputdirectory "")
@@
 			(at 2.975 -1.8 180)
 			(layer "F.SilkS")
+			(hide yes)
 			(effects
 				(font
@@
 			(at 0 -1.85 0)
 			(layer "F.SilkS")
+			(hide yes)
 			(effects
 				(font
@@
 	)
 	(segment
-		(start 116.8695 235.046)
-		(end 116.8695 252.806)
+		(start 134.5655 176.53)
+		(end 276.0535 176.53)
 		(width 0.2)
 		(layer "B.Cu")
@@
 	)
 	(segment
-		(start 117.1695 193.926)
-		(end 133.4195 177.676)
+		(start 278.3395 178.816)
+		(end 290.068 178.816)
 		(width 0.2)
 		(layer "B.Cu")
@@
 	)
 	(segment
-		(start 115.7495 193.926)
-		(end 117.1695 193.926)
+		(start 116.8695 235.046)
+		(end 116.8695 252.806)
 		(width 0.2)
 		(layer "B.Cu")
@@
 	)
 	(segment
-		(start 277.1995 177.676)
-		(end 278.3395 178.816)
+		(start 116.8695 252.806)
+		(end 115.7495 253.926)
 		(width 0.2)
 		(layer "B.Cu")
@@
 	)
 	(segment
-		(start 116.8695 252.806)
-		(end 115.7495 253.926)
+		(start 276.0535 176.53)
+		(end 278.3395 178.816)
 		(width 0.2)
 		(layer "B.Cu")
@@
 	)
 	(segment
+		(start 117.1695 193.926)
+		(end 134.5655 176.53)
+		(width 0.2)
+		(layer "B.Cu")
+		(net 6)
+	)
+	(segment
 		(start 116.8695 232.806)
 		(end 115.7495 233.926)
@@
 	)
 	(segment
-		(start 278.3395 178.816)
-		(end 290.068 178.816)
-		(width 0.2)
-		(layer "B.Cu")
-		(net 6)
-	)
-	(segment
-		(start 133.4195 177.676)
-		(end 277.1995 177.676)
+		(start 116.9495 195.126)
+		(end 116.9495 212.726)
 		(width 0.2)
 		(layer "B.Cu")
@@
 	)
 	(segment
-		(start 116.9495 195.126)
-		(end 116.9495 212.726)
+		(start 115.7495 193.926)
+		(end 117.1695 193.926)
 		(width 0.2)
 		(layer "B.Cu")
@@
 	)
 	(segment
-		(start 276.8095 192.526)
-		(end 278.3395 194.056)
+		(start 235.7495 193.926)
+		(end 237.1495 192.526)
 		(width 0.2)
 		(layer "B.Cu")
@@
 	)
 	(segment
-		(start 235.8295 233.926)
-		(end 236.8695 232.886)
+		(start 274.32 192.786)
+		(end 288.798 192.786)
 		(width 0.2)
 		(layer "B.Cu")
@@
 	)
 	(segment
-		(start 236.8695 195.046)
-		(end 235.7495 193.926)
+		(start 235.8295 233.926)
+		(end 236.8695 232.886)
 		(width 0.2)
 		(layer "B.Cu")
@@
 	)
 	(segment
-		(start 237.1495 192.526)
-		(end 276.8095 192.526)
+		(start 236.8695 195.046)
+		(end 235.7495 193.926)
 		(width 0.2)
 		(layer "B.Cu")
@@
 	)
 	(segment
-		(start 235.7495 193.926)
-		(end 237.1495 192.526)
+		(start 274.06 192.526)
+		(end 274.32 192.786)
 		(width 0.2)
 		(layer "B.Cu")
@@
 	)
 	(segment
-		(start 278.3395 194.056)
+		(start 237.1495 192.526)
+		(end 274.06 192.526)
+		(width 0.2)
+		(layer "B.Cu")
+		(net 11)
+	)
+	(segment
+		(start 288.798 192.786)
 		(end 290.068 194.056)
 		(width 0.2)
@@
 	)
 	(segment
-		(start 216.9495 232.726)
-		(end 215.7495 233.926)
+		(start 217.4695 192.126)
+		(end 271.424 192.126)
 		(width 0.2)
 		(layer "B.Cu")
@@
 	)
 	(segment
-		(start 251.215532 189.98)
-		(end 276.8035 189.98)
+		(start 216.9495 232.726)
+		(end 215.7495 233.926)
 		(width 0.2)
 		(layer "B.Cu")
@@
 	)
 	(segment
-		(start 228.6995 187.456)
-		(end 229.2595 188.016)
+		(start 273.304 190.246)
+		(end 288.798 190.246)
 		(width 0.2)
 		(layer "B.Cu")
@@
 	)
 	(segment
-		(start 235.0795 188.016)
-		(end 235.6395 187.456)
-		(width 0.2)
-		(layer "B.Cu")
-		(net 44)
-	)
-	(segment
-		(start 248.691532 187.456)
-		(end 251.215532 189.98)
+		(start 271.424 192.126)
+		(end 273.304 190.246)
 		(width 0.2)
 		(layer "B.Cu")
@@
 	)
 	(segment
-		(start 215.6695 193.926)
-		(end 222.1395 187.456)
-		(width 0.2)
-		(layer "B.Cu")
-		(net 44)
-	)
-	(segment
-		(start 235.6395 187.456)
-		(end 248.691532 187.456)
-		(width 0.2)
-		(layer "B.Cu")
-		(net 44)
-	)
-	(segment
-		(start 278.3395 191.516)
-		(end 290.068 191.516)
-		(width 0.2)
-		(layer "B.Cu")
-		(net 44)
-	)
-	(segment
 		(start 216.8695 212.806)
 		(end 215.7495 213.926)
@@
 	)
 	(segment
-		(start 276.8035 189.98)
-		(end 278.3395 191.516)
-		(width 0.2)
-		(layer "B.Cu")
-		(net 44)
-	)
-	(segment
-		(start 222.1395 187.456)
-		(end 228.6995 187.456)
+		(start 215.6695 193.926)
+		(end 217.4695 192.126)
 		(width 0.2)
 		(layer "B.Cu")
@@
 	)
 	(segment
-		(start 229.2595 188.016)
-		(end 235.0795 188.016)
+		(start 288.798 190.246)
+		(end 290.068 191.516)
 		(width 0.2)
 		(layer "B.Cu")
@@
 	)
 	(segment
+		(start 358.5972 189.0522)
+		(end 363.5502 194.0052)
+		(width 0.2)
+		(layer "F.Cu")
+		(net 72)
+	)
+	(segment
+		(start 355.9442 189.0522)
+		(end 358.5972 189.0522)
+		(width 0.2)
+		(layer "F.Cu")
+		(net 72)
+	)
+	(segment
 		(start 352.0442 235.1992)
 		(end 353.2632 233.9802)
@@
 	)
 	(segment
+		(start 355.8642 209.0522)
+		(end 358.5612 209.0522)
+		(width 0.2)
+		(layer "F.Cu")
+		(net 74)
+	)
+	(segment
+		(start 358.5612 209.0522)
+		(end 363.4232 213.9142)
+		(width 0.2)
+		(layer "F.Cu")
+		(net 74)
+	)
+	(segment
 		(start 355.8642 229.0522)
 		(end 358.9002 229.0522)
@@
 	)
 	(segment
+		(start 355.7842 249.0522)
+		(end 358.5262 249.0522)
+		(width 0.2)
+		(layer "F.Cu")
+		(net 76)
+	)
+	(segment
+		(start 358.5262 249.0522)
+		(end 363.4232 253.9492)
+		(width 0.2)
+		(layer "F.Cu")
+		(net 76)
+	)
+	(segment
