File: pcb/pcb.kicad_pcb (KiCad board)
At the start: 2 copper layers, 386.1 x 84.1 mm, 138 parts, among them P1 L to R, P2 R to L, SW1 SW_SPST, SW10 SW_SPST, SW11 SW_SPST, SW12 SW_SPST, SW13 SW_SPST, SW14 SW_SPST, SW15 SW_SPST, SW16 SW_SPST, SW17 SW_SPST, SW18 SW_SPST, SW19 SW_SPST, SW2 SW_SPST, SW20 SW_SPST, SW21 SW_SPST, SW22 SW_SPST, SW23 SW_SPST, SW24 SW_SPST, SW25 SW_SPST, SW26 SW_SPST, SW27 SW_SPST, SW28 SW_SPST, SW29 SW_SPST, SW3 SW_SPST, SW30 SW_SPST, SW31 SW_SPST, SW32 SW_SPST, SW33 SW_SPST, SW34 SW_SPST, SW35 SW_SPST, SW36 SW_SPST, SW37 SW_SPST, SW38 SW_SPST, SW39 SW_SPST, SW4 SW_SPST, SW40 SW_SPST, SW41 SW_SPST, SW42 SW_SPST, SW43 SW_SPST, SW44 SW_SPST, SW45 SW_SPST, SW46 SW_SPST, SW47 SW_SPST, SW48 SW_SPST, SW49 SW_SPST, SW5 SW_SPST, SW50 SW_SPST, SW51 SW_SPST, SW52 SW_SPST, SW53 SW_SPST, SW54 SW_SPST, SW55 SW_SPST, SW56 SW_SPST, SW57 SW_SPST, SW58 SW_SPST, SW59 SW_SPST, SW6 SW_SPST, SW60 SW_SPST, SW61 SW_SPST, SW62 SW_SPST, SW63 SW_SPST, SW64 SW_SPST, SW7 SW_SPST, SW8 SW_SPST, SW9 SW_SPST, U1 RP2040-ZERO, U2 RP2040-ZERO

Commit message: to low prof
Parts:
- SW1, SW10, SW11, SW12, SW13, SW14, SW15, SW16, SW17, SW18, SW19, SW2, SW20, SW21, SW22, SW23, SW24, SW25, SW26, SW27, SW28, SW29, SW3, SW30, SW31, SW32, SW33, SW34, SW35, SW36, SW37, SW38, SW39, SW4, SW40, SW41, SW42, SW43, SW44, SW45, SW46, SW47, SW48, SW49, SW5, SW50, SW51, SW52, SW53, SW54, SW55, SW56, SW57, SW58, SW59, SW6, SW60, SW61, SW62, SW63, SW64, SW7, SW8, SW9: footprint Keyboard Footprints:SW_MX_THT_nSilk -> Keyboard Footprints:SW_Kailh_Choc_V2_THT
- moved D59 10.2 mm to (343.5, 194.0), turned to 180 degrees
Routing:
- net c0l: track 245.3 -> 0.00 mm
- net c0r: track 229.8 -> 0.00 mm
- net c1l: track 224.9 -> 0.00 mm
- net r3r: track 212.3 -> 0.00 mm
- net c1r: track 208.8 -> 0.00 mm
- net c2l: track 206.5 -> 0.00 mm
- net r2r: track 195.8 -> 0.00 mm
- net r0r: track 194.1 -> 0.00 mm
- net c2r: track 190.7 -> 0.00 mm
- net c3l: track 185.8 -> 0.00 mm
- net r1r: track 183.7 -> 0.00 mm
- net c4l: track 169.8 -> 0.00 mm
- net c3r: track 165.6 -> 0.00 mm
- net c4r: track 144.3 -> 0.00 mm
- net c5l: track 139.3 -> 0.00 mm
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
Commit message: sv
Routing:
- net c0l: track 0.00 -> 243.0 mm
- net c1l: track 0.00 -> 222.1 mm
- net c2l: track 0.00 -> 200.9 mm
- net c3l: track 0.00 -> 180.0 mm
- net c4l: track 0.00 -> 159.0 mm
- net c5l: track 0.00 -> 138.8 mm
- net c6l: track 0.00 -> 117.9 mm
- net c7l: track 0.00 -> 98.0 mm
- net r3l: track 157.8 -> 225.2 mm
- net r2l: track 157.9 -> 206.6 mm
- net VCCL: track 0.00 -> 31.7 mm
- net GNDPWRL: track 0.00 -> 31.0 mm
- net r1l: track 157.8 -> 186.4 mm
- net r0l: track 157.9 -> 186.0 mm
- net SCL: track 0.00 -> 27.6 mm
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
Commit message: agh need to retrace some stuff will do tmmr
Parts:
- moved D12 10.1 mm to (483.5, 213.9), turned to 180 degrees
- moved D18 10.1 mm to (483.5, 234.0), turned to 180 degrees
- moved D24 10.1 mm to (483.5, 253.9), turned to 180 degrees
- moved D39 10.1 mm to (443.4, 194.0), turned to 180 degrees
- moved D40 10.1 mm to (443.4, 214.0), turned to 180 degrees
- moved D41 10.1 mm to (443.4, 234.0), turned to 180 degrees
- moved D42 10.1 mm to (443.4, 254.0), turned to 180 degrees
- moved D47 10.1 mm to (403.3, 194.0), turned to 180 degrees
- moved D48 10.1 mm to (403.3, 213.9), turned to 180 degrees
- moved D49 10.1 mm to (403.3, 234.0), turned to 180 degrees
- moved D50 10.1 mm to (403.3, 254.1), turned to 180 degrees
- moved D56 10.1 mm to (363.3, 213.9), turned to 180 degrees
- moved D57 10.1 mm to (363.3, 234.0), turned to 180 degrees
- moved D58 10.1 mm to (363.3, 253.9), turned to 180 degrees
- moved D6 10.1 mm to (483.5, 194.0), turned to 180 degrees
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Routing:
- net c0r: track 0.00 -> 239.7 mm
- net c1r: track 0.00 -> 217.7 mm
- net c2r: track 0.00 -> 198.6 mm
- net r0r: track 0.00 -> 196.7 mm
- net c3r: track 0.00 -> 175.5 mm
- net c4r: track 0.00 -> 154.2 mm
- net c5r: track 0.00 -> 133.2 mm
- net c6r: track 0.00 -> 114.5 mm
- net r3r: track 0.00 -> 94.9 mm
- net c7r: track 0.00 -> 93.1 mm
- net r2r: track 0.00 -> 65.3 mm
- net r1r: track 0.00 -> 41.3 mm
- net Net-(D54-A): track 0.00 -> 6.51 mm
- net Net-(D50-A): track 0.00 -> 6.40 mm
- net Net-(D64-A): track 0.00 -> 6.38 mm
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
Commit message: fix
Routing:
- net r1r: track 41.3 -> 199.1 mm
- net r2r: track 65.3 -> 220.8 mm
- net r3r: track 94.9 -> 244.7 mm
- net VCCR: track 0.00 -> 43.2 mm
- net SDA: track 20.3 -> 62.4 mm
- net GNDPWRR: track 0.00 -> 39.4 mm
- net SCL: track 27.6 -> 65.4 mm
- net c3r: track 175.5 -> 177.1 mm
- net c7r: track 93.1 -> 94.5 mm
Other:
- outline, holes or cut-outs redrawn
- board text added: "V001"
