File: pcb/pcb.kicad_pcb (KiCad board)
At the start: 2 copper layers, 386.1 x 84.1 mm, 138 parts, among them P1 L to R, P2 R to L, SW1 SW_SPST, SW10 SW_SPST, SW11 SW_SPST, SW12 SW_SPST, SW13 SW_SPST, SW14 SW_SPST, SW15 SW_SPST, SW16 SW_SPST, SW17 SW_SPST, SW18 SW_SPST, SW19 SW_SPST, SW2 SW_SPST, SW20 SW_SPST, SW21 SW_SPST, SW22 SW_SPST, SW23 SW_SPST, SW24 SW_SPST, SW25 SW_SPST, SW26 SW_SPST, SW27 SW_SPST, SW28 SW_SPST, SW29 SW_SPST, SW3 SW_SPST, SW30 SW_SPST, SW31 SW_SPST, SW32 SW_SPST, SW33 SW_SPST, SW34 SW_SPST, SW35 SW_SPST, SW36 SW_SPST, SW37 SW_SPST, SW38 SW_SPST, SW39 SW_SPST, SW4 SW_SPST, SW40 SW_SPST, SW41 SW_SPST, SW42 SW_SPST, SW43 SW_SPST, SW44 SW_SPST, SW45 SW_SPST, SW46 SW_SPST, SW47 SW_SPST, SW48 SW_SPST, SW49 SW_SPST, SW5 SW_SPST, SW50 SW_SPST, SW51 SW_SPST, SW52 SW_SPST, SW53 SW_SPST, SW54 SW_SPST, SW55 SW_SPST, SW56 SW_SPST, SW57 SW_SPST, SW58 SW_SPST, SW59 SW_SPST, SW6 SW_SPST, SW60 SW_SPST, SW61 SW_SPST, SW62 SW_SPST, SW63 SW_SPST, SW64 SW_SPST, SW7 SW_SPST, SW8 SW_SPST, SW9 SW_SPST, U1 RP2040-ZERO, U2 RP2040-ZERO

Commit message: wahoo
Parts:
- moved C1 20.1 mm to (286.0, 188.3)
- moved C2 20.1 mm to (286.0, 184.3)
- moved R2 20.1 mm to (286.0, 192.1)
- moved P1 19.7 mm to (288.8, 179.3)
- moved U1 12.6 mm to (270.0, 187.3)
Routing:
- net SDA: track 62.4 -> 83.8 mm
- net GNDPWRL: track 31.0 -> 51.1 mm
- net VCCL: track 31.7 -> 46.3 mm
- net r0l: track 185.0 -> 171.8 mm
- net c7l: track 98.0 -> 85.2 mm
- net c6l: track 117.9 -> 105.9 mm
- net SCL: track 65.4 -> 76.9 mm
- net r1l: track 186.4 -> 175.0 mm
- net r3l: track 227.9 -> 217.2 mm
- net r2l: track 205.8 -> 196.2 mm
- net c0l: track 243.0 -> 234.9 mm
- net c1l: track 222.1 -> 214.8 mm
- net c2l: track 200.9 -> 206.2 mm
- net c5l: track 138.8 -> 134.8 mm
- net c4l: track 159.0 -> 157.1 mm
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